File: V3/ir_beacon.sch (EAGLE design)
At the start: 35 parts, among them J2 B-, J3 B+, SW1 CNK-L202_MS02, U1 555_TIMER_DIP8

Commit message: Changed the testpoint type slightly, added a few more to the board. Moved around some traces and added many more vias for thermal conductivity. Generated new gerbers for the beacon board.
Parts:
- added TP4: LED-, meltylib:TESTPOINT_A
- added TP5: LED+, meltylib:TESTPOINT_A
- C2, C3, C4, C5: device jack_RCL:CAP_SMD -> jack_RCL:CAP_SMD_0805
- R1, R2, R4: device jack_RCL:RES_SMD0805 -> jack_RCL:RES_SMD_0805
- R3: device jack_RCL:RES_SMD1206 -> jack_RCL:RES_SMD_1206
- TP1, TP2, TP3: device jack_electromechanical:TEST_POINT -> meltylib:TESTPOINT_A
Connections:
- net 555CAP: now also TP3.TP; no longer TP3.P
- net GND: now also TP2.TP; no longer TP2.P
- net N$11: now also TP4.TP
- net N$16: now also TP1.TP; no longer TP1.P
- net V_BATT: now also TP5.TP
Other:
- moved on the sheet: Q1, TP1
